File: skill_test/skill_test.brd (EAGLE design)
At the start: 100 x 50 mm, 36 parts, among them Q1 16Mhz

Commit message: Fixed pin mapping from ESP
Parts:
- removed R8: 10k, rcl:0204/7
Connections:
- removed net N$9: R8.2, U$1.13
- new net SS: U$1.13, U$3.7
- net GND: no longer R8.1
Routing:
- net N$9: track 16.6 -> 0.00 mm
- net SS: track 0.00 -> 9.31 mm
- net GND: track 292.4 -> 293.0 mm
Changed lines of the file:
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@@
 <attribute name="SPICEPREFIX" value="R" x="158.8" y="-51.1" size="1.778" layer="27" display="off"/>
-</element>
-<element name="R8" library="rcl" library_urn="urn:adsk.eagle:library:334" package="0204/7" package3d_urn="urn:adsk.eagle:package:23498/2" value="10k" x="53.39" y="10.98" smashed="yes" rot="R270">
-<attribute name="NAME" x="52.9854" y="10.12" size="0.9906" layer="25" ratio="10" rot="R270"/>
-<attribute name="POPULARITY" value="48" x="-44.4" y="-6.8" size="1.778" layer="27" rot="R270" display="off"/>
-<attribute name="SPICEPREFIX" value="R" x="-44.4" y="-6.8" size="1.778" layer="27" rot="R270" display="off"/>
 </element>
 <element name="R9" library="rcl" library_urn="urn:adsk.eagle:library:334" package="0204/7" package3d_urn="urn:adsk.eagle:package:23498/2" value="10k" x="61.69" y="11.04" smashed="yes" rot="R270">
@@
 <contactref element="ESPSERIAL" pad="4"/>
 <contactref element="BOOTOPTION" pad="2"/>
-<contactref element="R8" pad="1"/>
 <contactref element="C4" pad="2"/>
 <contactref element="U$6" pad="4"/>
@@
 <wire x1="24.63" y1="12.4" x2="24.6" y2="12.43" width="0.381" layer="16"/>
 <wire x1="32.2" y1="26.01" x2="32.2" y2="17.9" width="0.381" layer="16"/>
-<wire x1="53.39" y1="14.79" x2="55.91" y2="14.79" width="0.381" layer="16"/>
-<wire x1="55.91" y1="14.79" x2="57.6" y2="13.1" width="0.381" layer="16"/>
 <wire x1="57.6" y1="13.1" x2="57.6" y2="10.48" width="0.381" layer="16"/>
-<wire x1="51.3199" y1="7.743971875" x2="51.3199" y2="12.7199" width="0.381" layer="16"/>
-<wire x1="51.3199" y1="12.7199" x2="53.39" y2="14.79" width="0.381" layer="16"/>
-<wire x1="50.042428125" y1="6.4665" x2="51.3199" y2="7.743971875" width="0.381" layer="16"/>
-<wire x1="46.8735" y1="6.4665" x2="50.042428125" y2="6.4665" width="0.381" layer="16"/>
+<wire x1="46.8735" y1="6.4665" x2="53.5865" y2="6.4665" width="0.381" layer="16"/>
 <wire x1="45.72" y1="25.4" x2="45.72" y2="25.4735" width="0.381" layer="16"/>
 <wire x1="45.72" y1="25.4735" x2="46.8" y2="26.5535" width="0.381" layer="16"/>
 <wire x1="46.8" y1="26.5535" x2="50.2465" y2="26.5535" width="0.381" layer="16"/>
-<wire x1="53.39" y1="23.41" x2="53.39" y2="14.79" width="0.381" layer="16"/>
-<wire x1="50.2465" y1="26.5535" x2="53.39" y2="23.41" width="0.381" layer="16"/>
 <polygon width="0.381" layer="16">
 <vertex x="101.1" y="50.9"/>
@@
 <via x="80.4" y="10.1" extent="1-16" drill="0.35"/>
 <via x="94.6" y="3.6" extent="1-16" drill="0.35"/>
+<wire x1="53.5865" y1="6.4665" x2="57.6" y2="10.48" width="0.381" layer="16"/>
+<wire x1="57.6" y1="19.2" x2="57.6" y2="10.48" width="0.381" layer="16"/>
+<wire x1="50.2465" y1="26.5535" x2="57.6" y2="19.2" width="0.381" layer="16"/>
 </signal>
 <signal name="UCC" class="2">
@@
 <contactref element="U$1" pad="14"/>
 <contactref element="U$3" pad="9"/>
-<wire x1="42.1" y1="13.93" x2="44.41" y2="13.93" width="0.381" layer="1"/>
-<wire x1="44.41" y1="13.93" x2="45.72" y2="15.24" width="0.381" layer="1"/>
+<wire x1="42.1" y1="13.93" x2="44.11" y2="13.93" width="0.381" layer="1"/>
+<wire x1="45.42" y1="15.24" x2="45.72" y2="15.24" width="0.381" layer="1"/>
+<wire x1="45.42" y1="15.24" x2="44.11" y2="13.93" width="0.381" layer="1"/>
 </signal>
 <signal name="N$10">
@@
 <wire x1="39.39" y1="7.926025" x2="40.882975" y2="9.419" width="0.508" layer="16"/>
 </signal>
-<signal name="N$9">
+<signal name="SS">
+<contactref element="U$3" pad="7"/>
+<wire x1="45.193225" y1="13.905" x2="46.1901375" y2="13.905" width="0.3048" layer="1"/>
+<wire x1="46.1901375" y1="13.905" x2="46.955" y2="14.6698625" width="0.3048" layer="1"/>
+<wire x1="46.955" y1="14.6698625" x2="46.955" y2="16.0101375" width="0.3048" layer="1"/>
+<wire x1="45.72" y1="17.2451375" x2="45.72" y2="17.78" width="0.3048" layer="1"/>
+<wire x1="46.955" y1="16.0101375" x2="45.72" y2="17.2451375" width="0.3048" layer="1"/>
+<wire x1="42.165" y1="12.495" x2="43.783225" y2="12.495" width="0.3048" layer="1"/>
+<wire x1="43.783225" y1="12.495" x2="45.193225" y2="13.905" width="0.3048" layer="1"/>
 <contactref element="U$1" pad="13"/>
-<contactref element="R8" pad="2"/>
-<wire x1="53.39" y1="7.17" x2="53.39" y2="7.16" width="0.381" layer="16"/>
-<wire x1="42.1" y1="12.43" x2="42.6015" y2="11.9285" width="0.381" layer="1"/>
-<wire x1="42.6015" y1="11.9285" x2="42.83811875" y2="11.9285" width="0.381" layer="1"/>
-<wire x1="42.83811875" y1="11.9285" x2="43.4" y2="11.36661875" width="0.381" layer="1"/>
-<wire x1="43.4" y1="11.36661875" x2="43.4" y2="7.2" width="0.381" layer="1"/>
-<wire x1="43.4" y1="7.2" x2="44.197890625" y2="6.402109375" width="0.381" layer="1"/>
-<wire x1="44.197890625" y1="6.402109375" x2="44.19878125" y2="6.403" width="0.254" layer="1"/>
-<wire x1="44.19878125" y1="6.403" x2="47.98121875" y2="6.403" width="0.254" layer="1"/>
-<wire x1="47.98121875" y1="6.403" x2="47.98421875" y2="6.4" width="0.254" layer="1"/>
-<wire x1="47.98421875" y1="6.4" x2="49.5" y2="6.4" width="0.254" layer="1"/>
-<wire x1="49.5" y1="6.4" x2="52.62" y2="6.4" width="0.381" layer="1"/>
-<wire x1="52.62" y1="6.4" x2="53.39" y2="7.17" width="0.381" layer="1"/>
+<wire x1="42.1" y1="12.43" x2="42.165" y2="12.495" width="0" layer="19" extent="1-1"/>
 </signal>
 <signal name="N$13">
